File: hardware/combined/cellguard_combined.kicad_sch (KiCad schematic)
At the start: 23 parts, among them J1 Raspberry Pi 5 GPIO Header, J2 ZY12PDN PD Trigger (5V), J3 ATORCH BW150 부하 입력, K1 4CH Relay [SZH-RLBG-012], U1 INA226 [VLT-VCM029], U2 Battery Babysitter [PRT-13777], U3 MLX90614 #1 (0x5A, 셀 중앙 / 모드 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, U4 ADS1115 [VLT-AD004], U5 DS18B20 #1 (셀 하단, 모드 1 전용), U6 TFT 3.5in SPI 480x320 V1.0, U7 DS18B20 #2 (셀 중앙, 모드 1 전용), U8 DS18B20 #3 (셀 단자쪽, 모드 1 전용), U9 MLX90614 #2 (0x5B, 셀 단자쪽 / 모드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

Commit message: docs(hardware): carry two mode 1 schematic notes into combined
모드 1 회로도에만 있던 두 가지를 통합 회로도로 옮겼다. 통합 회로는 모드 1을
그대로 포함하므로 이 둘이 빠지면 mode1 회로도를 계속 곁눈질해야 한다.

- CH3을 열었을 때의 정상 동작. 모드 1은 0x55가 버스에서 사라지고 모드 2는
  팩이 무부하로 꺼져 INA226이 0V를 읽는다 — 둘 다 고장이 아니다.
- 온도 다점 측정의 최댓값 규칙과 DS18B20 Skip ROM 동시 변환(750ms).

Co-Authored-By: Claude Opus 5 <noreply@anthropic.com>
Claude-Session: https://claude.ai/code/session_01GJZ3iq4n6rFBxLGAgZh4q9
Other:
- note added: "DS18B20 3개는 같은 3선에 병렬로 문다. 1-Wire 고유 64비트 ROM 코드라 주소 설정이 필요 없고,"
- note added: "INA226 은 Pi 3.3V 로 동작하므로 모드 1 에서는 마스터 차단 후에도 셀 전압 감시가 계속된다."
- note added: "Skip ROM + Convert T 로 셋을 동시에 변환해 개수가 늘어도 750ms 그대로다(순차로 하면 2250ms)."
- note added: "[주의] CH3 을 열면 두 모드 다 측정 대상이 완전히 분리된다 — 아래는 고장이 아니라 정상 동작이다."
- note added: "temp_ir_surface = max(#1, #2) temp_contact = max(DS18B20 #1, #2, #3)"
- note added: "모드 1: BQ27441 이 꺼져 I2C 0x55 가 버스에서 사라진다. 릴레이 상태를 조건으로 걸지 않으면 센서 오류 알림이 폭주한다."
- note added: "모드 2: 팩이 무부하가 되어 스스로 꺼지므로 INA226 이 0V 를 읽는다. 배터리 사망으로 오독하지 마라."
- note added: "온도는 다점 측정이고 쓰는 값은 최댓값이다 — 열폭주는 국부에서 시작하므로 평균을 쓰면 초기 신호가 희석된다."

Commit message: docs: measure room temperature and define heat rise (surface - ambient)
Plan change 2026-09-25: reverses the "temp_ambient is not measured"
decision. Mode 1 repurposes MLX90614 #2 (0x5B) from the cell terminal
zone to room temperature (Ta register recommended, verify as H10); the
cell IR becomes one zone and the terminal hot spot is covered by the
terminal DS18B20. Mode 2 uses one DS18B20 as the room probe (which probe
in the combined rig is left as 정의 필요).

Heat rise = representative surface temp - ambient. AI T_rise feature,
mode 2 thermal slope on heat rise, and dashboard tempAmbientC/heatRiseC
are recorded as decided direction but not implemented. Schematic labels
regenerated (ERC 0, nets unchanged); SVGs left as-is because they were
already stale and re-export is a 400k-line unrelated diff.

Co-Authored-By: Claude Opus 5.5 <noreply@anthropic.com>
Parts:
- U9: value MLX90614 #2 (0x5B, 셀 단자쪽 / 모드 2: USB-A 포트쪽) -> MLX90614 #2 (0x5B, 모드 1: 실온 / 모드 2: USB-A 포트쪽)
Other:
- note added: "0x5B MLX90614 #2 모드 1 실온(Ta) / 모드 2 IR 표면온도 (EEPROM 0x0E 로 주소 변경한 개체)"
- note added: "temp_ambient MLX #2 (Ta) DS18B20 1개 실온. 셀·팩·BW150 에서 10cm 이상 떨어뜨린다"
- note added: "temp_contact DS18B20 x3 null 보조배터리에 옮겨 붙이지 않는다 (실온 1개만 예외)"
- note added: "temp_ir_surface MLX #1 MLX x2 브래킷째 옮겨 겨눈다"
- note added: "모드 1: temp_ir_surface = #1 모드 2: max(#1, #2) temp_contact = max(DS18B20 #1, #2, #3)"
- note removed: "0x5B MLX90614 #2 IR 표면온도 (EEPROM 0x0E 로 주소 변경한 개체)"
- note removed: "temp_contact DS18B20 x3 null 보조배터리에 옮겨 붙이지 않는다"
- note removed: "temp_ir_surface = max(#1, #2) temp_contact = max(DS18B20 #1, #2, #3)"
- note removed: "temp_ir_surface MLX x2 MLX x2 브래킷째 옮겨 겨눈다"
Changed lines of the file:
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@@
 		(dnp no)
 		(property "Reference" "U9" (at 574.04 140.97 0) (effects (font (face "Apple SD Gothic Neo") (size 1.27 1.27)) (justify left bottom)))
-		(property "Value" "MLX90614 #2 (0x5B, 셀 단자쪽 / 모드 2: USB-A 포트쪽)" (at 574.04 143.51 0) (effects (font (face "Apple SD Gothic Neo") (size 1.27 1.27)) (justify left bottom)))
+		(property "Value" "MLX90614 #2 (0x5B, 모드 1: 실온 / 모드 2: USB-A 포트쪽)" (at 574.04 143.51 0) (effects (font (face "Apple SD Gothic Neo") (size 1.27 1.27)) (justify left bottom)))
 		(property "Footprint" "" (at 590.55 152.40 0) (effects (font (face "Apple SD Gothic Neo") (size 1.27 1.27)) (hide yes)))
 		(property "Datasheet" "" (at 590.55 152.40 0) (effects (font (face "Apple SD Gothic Neo") (size 1.27 1.27)) (hide yes)))
@@
 		(effects (font (face "Apple SD Gothic Neo") (size 2.0 2.0)) (justify left bottom))
 	)
-	(text "0x5B  MLX90614 #2  IR 표면온도          (EEPROM 0x0E 로 주소 변경한 개체)"
+	(text "0x5B  MLX90614 #2  모드 1 실온(Ta) / 모드 2 IR 표면온도  (EEPROM 0x0E 로 주소 변경한 개체)"
 		(exclude_from_sim no)
 		(at 300.00 557.40 0)
@@
 		(effects (font (face "Apple SD Gothic Neo") (size 2.0 2.0)) (justify left bottom))
 	)
-	(text "temp_ir_surface         MLX x2        MLX x2        브래킷째 옮겨 겨눈다"
+	(text "temp_ir_surface         MLX #1        MLX x2        브래킷째 옮겨 겨눈다"
 		(exclude_from_sim no)
 		(at 580.00 371.80 0)
 		(effects (font (face "Apple SD Gothic Neo") (size 2.0 2.0)) (justify left bottom))
 	)
-	(text "temp_contact            DS18B20 x3    null          보조배터리에 옮겨 붙이지 않는다"
+	(text "temp_ambient            MLX #2 (Ta)   DS18B20 1개   실온. 셀·팩·BW150 에서 10cm 이상 떨어뜨린다"
 		(exclude_from_sim no)
 		(at 580.00 377.00 0)
 		(effects (font (face "Apple SD Gothic Neo") (size 2.0 2.0)) (justify left bottom))
 	)
+	(text "temp_contact            DS18B20 x3    null          보조배터리에 옮겨 붙이지 않는다 (실온 1개만 예외)"
+		(exclude_from_sim no)
+		(at 580.00 382.20 0)
+		(effects (font (face "Apple SD Gothic Neo") (size 2.0 2.0)) (justify left bottom))
+	)
 	(text "pressure_raw            FSR 406       null          외장 케이스에 가려 부착 불가"
 		(exclude_from_sim no)
-		(at 580.00 382.20 0)
+		(at 580.00 387.40 0)
 		(effects (font (face "Apple SD Gothic Neo") (size 2.0 2.0)) (justify left bottom))
 	)
 	(text "soc_pct                 BQ27441       null          완제품이라 셀에 접근 불가"
 		(exclude_from_sim no)
-		(at 580.00 387.40 0)
+		(at 580.00 392.60 0)
 		(effects (font (face "Apple SD Gothic Neo") (size 2.0 2.0)) (justify left bottom))
 	)
 	(text "gas_raw / acoustic_raw  null          null          이 회로에 센서 자체가 없다"
 		(exclude_from_sim no)
-		(at 580.00 392.60 0)
+		(at 580.00 397.80 0)
 		(effects (font (face "Apple SD Gothic Neo") (size 2.0 2.0)) (justify left bottom))
 	)
 	(text "diag_phase / load_target_a  null      null          P0~P6 을 실행하지 않는 프로필이다"
 		(exclude_from_sim no)
-		(at 580.00 397.80 0)
+		(at 580.00 403.00 0)
 		(effects (font (face "Apple SD Gothic Neo") (size 2.0 2.0)) (justify left bottom))
 	)
 	(text "온도는 다점 측정이고 쓰는 값은 최댓값이다 — 열폭주는 국부에서 시작하므로 평균을 쓰면 초기 신호가 희석된다."
 		(exclude_from_sim no)
-		(at 580.00 403.00 0)
-		(effects (font (face "Apple SD Gothic Neo") (size 2.0 2.0)) (justify left bottom))
-	)
-	(text "  temp_ir_surface = max(#1, #2)      temp_contact = max(DS18B20 #1, #2, #3)"
-		(exclude_from_sim no)
 		(at 580.00 408.20 0)
 		(effects (font (face "Apple SD Gothic Neo") (size 2.0 2.0)) (justify left bottom))
 	)
+	(text "  모드 1: temp_ir_surface = #1   모드 2: max(#1, #2)   temp_contact = max(DS18B20 #1, #2, #3)"
+		(exclude_from_sim no)
+		(at 580.00 413.40 0)
+		(effects (font (face "Apple SD Gothic Neo") (size 2.0 2.0)) (justify left bottom))
+	)
 	(text "  DS18B20 3개는 같은 3선에 병렬로 문다. 1-Wire 고유 64비트 ROM 코드라 주소 설정이 필요 없고,"
 		(exclude_from_sim no)
-		(at 580.00 413.40 0)
+		(at 580.00 418.60 0)
 		(effects (font (face "Apple SD Gothic Neo") (size 2.0 2.0)) (justify left bottom))
 	)
 	(text "  Skip ROM + Convert T 로 셋을 동시에 변환해 개수가 늘어도 750ms 그대로다(순차로 하면 2250ms)."
 		(exclude_from_sim no)
-		(at 580.00 418.60 0)
+		(at 580.00 423.80 0)
 		(effects (font (face "Apple SD Gothic Neo") (size 2.0 2.0)) (justify left bottom))
 	)
 	(text "모드 2 IR 배치: 0x5A=케이스 중앙 / 0x5B=USB-A 출력 포트쪽. 표면에서 최대 5cm, 스팟 중심 4cm 이상 분리."
 		(exclude_from_sim no)
-		(at 580.00 423.80 0)
+		(at 580.00 429.00 0)
 		(effects (font (face "Apple SD Gothic Neo") (size 2.0 2.0)) (justify left bottom))
 	)
 	(text "[주의] 케이스 표면온도는 셀 온도가 아니다. 모드 1 의 55/60도 문턱을 모드 2 에 그대로 쓰지 마라."
 		(exclude_from_sim no)
-		(at 580.00 429.00 0)
+		(at 580.00 434.20 0)
 		(effects (font (face "Apple SD Gothic Neo") (size 2.0 2.0)) (justify left bottom))
 	)
 	(text "[!] MLX90614 는 두 모드가 공유하므로 마운트를 떼었다 붙일 수 있게 만든다"
 		(exclude_from_sim no)
-		(at 580.00 437.20 0)
+		(at 580.00 442.40 0)
 		(effects (font (face "Apple SD Gothic Neo") (size 2.5 2.5)) (justify left bottom))
 	)
 	(text "접착 고정이 아니라 나사 1개 또는 클램프로 각도·거리를 바꿀 수 있게 하고, 케이블에 여유를 준다."
 		(exclude_from_sim no)
-		(at 580.00 445.20 0)
+		(at 580.00 450.40 0)
 		(effects (font (face "Apple SD Gothic Neo") (size 2.0 2.0)) (justify left bottom))
 	)
 	(text "모드 1 부착 거리는 2cm 이내 — FOV 35도라 스팟 지름 = 0.63 x 거리, 18650(지름 1.8cm) 안에 들어와야 한다."
 		(exclude_from_sim no)
-		(at 580.00 450.40 0)
+		(at 580.00 455.60 0)
 		(effects (font (face "Apple SD Gothic Neo") (size 2.0 2.0)) (justify left bottom))
 	)
 	(text "둘 다 출고 시 0x5A 이므로 한 개씩 따로 연결해 U9 를 0x5B 로 바꾼다. EEPROM 쓰기에는 PEC 바이트가 필수다."
 		(exclude_from_sim no)
-		(at 580.00 455.60 0)
+		(at 580.00 460.80 0)
 		(effects (font (face "Apple SD Gothic Neo") (size 2.0 2.0)) (justify left bottom))
 	)
 	(text "출고 상태는 갱신 865ms + 스파이크 50% 감쇠다. EEPROM 0x25 를 IIR=100 / FIR=111 로 재설정 -> 95.2ms."
 		(exclude_from_sim no)
-		(at 580.00 460.80 0)
+		(at 580.00 466.00 0)
 		(effects (font (face "Apple SD Gothic Neo") (size 2.0 2.0)) (justify left bottom))
 	)
 	(text "[!] TFT 3.5in — 표시 전용 9핀만 쓴다"
 		(exclude_from_sim no)
-		(at 580.00 469.00 0)
+		(at 580.00 474.20 0)
 		(effects (font (face "Apple SD Gothic Neo") (size 2.5 2.5)) (justify left bottom))
 	)
 	(text "T_CLK / T_CS / T_DIN / T_DO / T_IRQ 5핀은 터치용, SDO(MISO)도 미결선."
 		(exclude_from_sim no)
-		(at 580.00 477.00 0)
+		(at 580.00 482.20 0)
 		(effects (font (face "Apple SD Gothic Neo") (size 2.0 2.0)) (justify left bottom))
 	)
 	(text "LED(백라이트)는 3.3V 직결 = 상시 점등.  VCC 는 3.3V — 안 켜지면 그때만 5V(물리핀 2·4)로 옮긴다."
 		(exclude_from_sim no)
-		(at 580.00 482.20 0)
+		(at 580.00 487.40 0)
 		(effects (font (face "Apple SD Gothic Neo") (size 2.0 2.0)) (justify left bottom))
 	)
 	(text "ILI9488 은 SPI 에서 RGB565 를 못 쓴다. 480x320 전체 갱신 약 460KB 이므로"
 		(exclude_from_sim no)
-		(at 580.00 487.40 0)
+		(at 580.00 492.60 0)
 		(effects (font (face "Apple SD Gothic Neo") (size 2.0 2.0)) (justify left bottom))
 	)
 	(text "100ms 계측 루프에 전체 화면 갱신을 올리지 마라 -> 부분 갱신 + 별도 스레드."
 		(exclude_from_sim no)
-		(at 580.00 492.60 0)
+		(at 580.00 497.80 0)
 		(effects (font (face "Apple SD Gothic Neo") (size 2.0 2.0)) (justify left bottom))
 	)
 	(text "모드 전환 절차 요약 (자세한 것은 통합 조립 가이드 8·9절)"
 		(exclude_from_sim no)
-		(at 580.00 500.80 0)
+		(at 580.00 506.00 0)
 		(effects (font (face "Apple SD Gothic Neo") (size 2.5 2.5)) (justify left bottom))
 	)
 	(text "모드 2 -> 모드 1:  BW150 0A/OFF -> pinctrl set 5,6,13,19 op dh -> USB-A 플러그를 보조배터리에서 뽑기"
 		(exclude_from_sim no)
-		(at 580.00 508.80 0)
+		(at 580.00 514.00 0)
 		(effects (font (face "Apple SD Gothic Neo") (size 2.0 2.0)) (justify left bottom))
 	)
 	(text "                   -> Pi·ZY12PDN 전원 분리 -> VBUS 를 SOURCE_P 에서 분리·절연 -> 셀 홀더 + 체결."
 		(exclude_from_sim no)
-		(at 580.00 514.00 0)
+		(at 580.00 519.20 0)
 		(effects (font (face "Apple SD Gothic Neo") (size 2.0 2.0)) (justify left bottom))
 	)
 	(text "모드 1 -> 모드 2:  BW150 0A/OFF -> CH1·CH2·CH3 OFF -> Pi·ZY12PDN 전원 분리 -> 셀을 홀더에서 빼기"
 		(exclude_from_sim no)
-		(at 580.00 519.20 0)
+		(at 580.00 524.40 0)
 		(effects (font (face "Apple SD Gothic Neo") (size 2.0 2.0)) (justify left bottom))
 	)
 	(text "                   -> 홀더 + 분리·절연 -> VBUS 체결 -> Pi 만 부팅 -> CH3 OFF 에서 CH4 ON -> 50ms 대기"
 		(exclude_from_sim no)
-		(at 580.00 524.40 0)
+		(at 580.00 529.60 0)
 		(effects (font (face "Apple SD Gothic Neo") (size 2.0 2.0)) (justify left bottom))
 	)
 	(text "                   -> 보조배터리 연결 -> 무부하 검산 -> BW150 0.1A 설정 -> CH3 ON -> BW150 출력 ON."
 		(exclude_from_sim no)
-		(at 580.00 529.60 0)
+		(at 580.00 534.80 0)
 		(effects (font (face "Apple SD Gothic Neo") (size 2.0 2.0)) (justify left bottom))
 	)
 	(text "무부하 통과 기준:  CAL=0x0A00, MFG=0x5449, DIE=0x2260, OVF=0, |current_a| <= 0.02A."
 		(exclude_from_sim no)
-		(at 580.00 534.80 0)
+		(at 580.00 540.00 0)
 		(effects (font (face "Apple SD Gothic Neo") (size 2.0 2.0)) (justify left bottom))
 	)
 	(text "PCB 없음 — 기성 모듈 + 배선 하네스다.  전력 경로는 0.75SQ 실리콘 배선, JD_VCC 만 점퍼선."
 		(exclude_from_sim no)
-		(at 580.00 543.00 0)
+		(at 580.00 548.20 0)
 		(effects (font (face "Apple SD Gothic Neo") (size 2.0 2.0)) (justify left bottom))
 	)
 	(text "예비품 없음: DS18B20 3개와 MLX90614 2개를 전부 투입했다. 고장 시 교체품이 없다."
 		(exclude_from_sim no)
-		(at 580.00 548.20 0)
-		(effects (font (face "Apple SD Gothic Neo") (size 2.0 2.0)) (justify left bottom))
-	)
+		(at 580.00 553.40 0)
+		(effects (font (face "Apple SD Gothic Neo") (size 2.0 2.0)) (justify left bottom))
+	)
