File: hardware/mode1/cellguard_mode1.kicad_sch (KiCad schematic)
At the start: 21 parts, among them J1 Raspberry Pi 5 GPIO Header, J2 ZY12PDN PD Trigger (5V), J3 ATORCH BW150 부하 입력, K1 4CH Relay [SZH-RLBG-012], U1 INA226 [VLT-VCM029], U2 Battery Babysitter [PRT-13777], U3 MLX90614 #1 (0x5A, 셀 중앙), U4 ADS1115 [VLT-AD004], U5 DS18B20 #1 (셀 하단), U6 OLED 0.96in SPI [CN0219], U7 DS18B20 #2 (셀 중앙), U8 DS18B20 #3 (셀 상단·단자쪽), U9 MLX90614 #2 (0x5B, 셀 단자쪽)

Commit message: feat(mode1): 현장 표시 화면을 0.96" OLED에서 3.5" TFT SPI 480x320(ILI9488)로 교체
14핀 모듈이지만 터치는 쓰지 않아 T_CLK/T_CS/T_DIN/T_DO/T_IRQ 5핀과
SDO(MISO)는 미결선이다. 표시용 SPI 5가닥(CS/RESET/DC-RS/SDI/SCK)의 GPIO는
구 OLED와 1:1로 같고, LED(백라이트) → 3.3V 한 가닥만 늘었다.

- 회로도: OLED 심볼을 TFT35(14핀)로 교체, 네트 OLED_RES/OLED_DC →
  TFT_RES/TFT_DC. 심볼이 길어져 우측 열 순서를 TFT-MLX-ADS-풀업으로
  재배치(R6가 주석 블록과 겹치는 것 방지). ERC 위반 0건, 넷리스트 확인.
- 새 gotcha 2건: ILI9488은 SPI에서 RGB565가 안 되고 픽셀당 3바이트(RGB666)라
  전체 화면 갱신 460KB → 100ms 계측 루프에 올리면 안 된다. VCC는 3.3V로
  넣되 보드에 LDO가 얹힌 개체는 안 켜질 수 있어 실물 확인 항목 H9 신설.
- 조립 작업서 STEP 8 전면 개정, STEP 16에 백라이트 점등 확인(H9) 추가,
  §7-1 인계표·부록 B 핀맵 갱신.

Co-Authored-By: Claude Opus 5 <noreply@anthropic.com>
Claude-Session: https://claude.ai/code/session_014zci1RutLJwRDUxRGnv1aB
Parts:
- U6: value OLED 0.96in SPI [CN0219] -> TFT 3.5in SPI 480x320 V1.0; symbol cellguard:OLED -> cellguard:TFT35
Connections:
- net +3V3: now also U6.1 (VCC), U6.8 (LED); no longer U6.2 (VCC)
- net GND: now also U6.2 (GND); no longer U6.1 (GND)
- net SPI_CE0: now also U6.3 (CS); no longer U6.7 (CS)
- net SPI_MOSI: now also U6.6 (SDI); no longer U6.4 (D1)
- net SPI_SCLK: now also U6.7 (SCK); no longer U6.3 (D0)
- net OLED_DC renamed TFT_DC
- net TFT_DC: now also U6.5 (DC/RS); no longer U6.6 (DC)
- net OLED_RES renamed TFT_RES
- net TFT_RES: now also U6.4 (RESET); no longer U6.5 (RES)
- no-connect marks 29 -> 35
Other:
- note added: "14핀 중 T_CLK / T_CS / T_DIN / T_DO / T_IRQ 5핀은 터치용이라 미결선."
- note added: "480x320 전체 갱신이 약 460KB 다. 100ms 계측 루프에 전체 화면 갱신을"
- note added: "LED(백라이트)는 3.3V 직결 = 상시 점등. 밝기 제어를 원하면 PWM GPIO 로 옮긴다."
- note added: "SDO(MISO)도 화면에서 읽을 일이 없어 미결선 -> SPI0 은 MOSI 단방향이다."
- note added: "SPI 배선 5가닥(CS/RESET/DC/SDI/SCK)은 교체 전 OLED와 GPIO가 완전히 같다."
- note added: "[!] TFT 3.5in — 표시 전용 9핀만 쓴다"
- note added: "[주의] ILI9488 은 SPI 에서 RGB565 를 못 쓴다. 픽셀당 3바이트(RGB666)라"
- note added: "[주의] VCC 는 3.3V 로 넣는다. 보드에 3.3V LDO 가 얹힌 개체는 3.3V 입력으로"
- note added: "드롭아웃이 모자라 화면이 안 켜질 수 있다 -> 그때만 5V(물리핀 2·4)로 옮긴다."
- note added: "로직(CS/SCK/SDI/DC/RESET)은 어느 쪽이든 3.3V TTL 이다."
- note added: "물리핀 1, 17 3.3V 센서 · TFT(VCC+LED) · 릴레이 VCC(옵토측)"
- note added: "물리핀 18 GPIO24 TFT RESET"
- note added: "물리핀 19 GPIO10 TFT SDI (MOSI)"
- note added: "물리핀 22 GPIO25 TFT DC/RS"
- note added: "물리핀 23 GPIO11 TFT SCK"
- note added: "물리핀 24 GPIO8 TFT CS (SPI0 CE0)"
- note added: "올리지 마라 -> 바뀐 영역만 부분 갱신하고, 표시는 계측과 별도 스레드로."
- note removed: "물리핀 1, 17 3.3V 센서 · OLED · 릴레이 VCC(옵토측)"
- note removed: "물리핀 18 GPIO24 OLED RES"
- note removed: "물리핀 19 GPIO10 OLED D1 (MOSI)"
- note removed: "물리핀 22 GPIO25 OLED DC"
- note removed: "물리핀 23 GPIO11 OLED D0 (SCLK)"
- note removed: "물리핀 24 GPIO8 OLED CS (SPI0 CE0)"
- moved on the sheet: U3, U4, U9

Commit message: docs: measure room temperature and define heat rise (surface - ambient)
Plan change 2026-09-25: reverses the "temp_ambient is not measured"
decision. Mode 1 repurposes MLX90614 #2 (0x5B) from the cell terminal
zone to room temperature (Ta register recommended, verify as H10); the
cell IR becomes one zone and the terminal hot spot is covered by the
terminal DS18B20. Mode 2 uses one DS18B20 as the room probe (which probe
in the combined rig is left as 정의 필요).

Heat rise = representative surface temp - ambient. AI T_rise feature,
mode 2 thermal slope on heat rise, and dashboard tempAmbientC/heatRiseC
are recorded as decided direction but not implemented. Schematic labels
regenerated (ERC 0, nets unchanged); SVGs left as-is because they were
already stale and re-export is a 400k-line unrelated diff.

Co-Authored-By: Claude Opus 5.5 <noreply@anthropic.com>
Parts:
- U9: value MLX90614 #2 (0x5B, 셀 단자쪽) -> MLX90614 #2 (0x5B, 실온 - 셀을 겨누지 않음)
Other:
- note added: "0x5B MLX90614 #2 실온 (Ta) - 셀·발열체에서 10cm 이상 (EEPROM 0x0E 로 주소 변경한 개체)"
- note added: "[!] MLX90614 #1 부착 거리 — 2cm 이내"
- note added: "temp_ir_surface = #1 temp_contact = max(DS18B20 #1, #2, #3) temp_ambient = #2 Ta"
- note added: "셀 IR 은 #1 한 존이고, #2 는 실온을 잰다 -> 발열값 = 표면온도 - 실온 (2026-09-25)."
- note removed: "0x5B MLX90614 #2 IR 표면온도 - 셀 단자쪽 (EEPROM 0x0E 로 주소 변경한 개체)"
- note removed: "MLX90614 소자 1개는 FOV 안의 '평균'만 낸다. 그래서 2개를 다른 지점에 겨눠 공간 피크를 만든다."
- note removed: "[!] MLX90614 부착 거리 — 2cm 이내"
- note removed: "temp_ir_surface = max(#1, #2) temp_contact = max(DS18B20 #1, #2, #3)"
Changed lines of the file:
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@@
 		(dnp no)
 		(property "Reference" "U9" (at 574.04 140.97 0) (effects (font (face "Apple SD Gothic Neo") (size 1.27 1.27)) (justify left bottom)))
-		(property "Value" "MLX90614 #2 (0x5B, 셀 단자쪽)" (at 574.04 143.51 0) (effects (font (face "Apple SD Gothic Neo") (size 1.27 1.27)) (justify left bottom)))
+		(property "Value" "MLX90614 #2 (0x5B, 실온 - 셀을 겨누지 않음)" (at 574.04 143.51 0) (effects (font (face "Apple SD Gothic Neo") (size 1.27 1.27)) (justify left bottom)))
 		(property "Footprint" "" (at 590.55 152.40 0) (effects (font (face "Apple SD Gothic Neo") (size 1.27 1.27)) (hide yes)))
 		(property "Datasheet" "" (at 590.55 152.40 0) (effects (font (face "Apple SD Gothic Neo") (size 1.27 1.27)) (hide yes)))
@@
 		(effects (font (face "Apple SD Gothic Neo") (size 2.0 2.0)) (justify left bottom))
 	)
-	(text "0x5B   MLX90614 #2  IR 표면온도 - 셀 단자쪽 (EEPROM 0x0E 로 주소 변경한 개체)"
+	(text "0x5B   MLX90614 #2  실온 (Ta) - 셀·발열체에서 10cm 이상 (EEPROM 0x0E 로 주소 변경한 개체)"
 		(exclude_from_sim no)
 		(at 300.00 391.40 0)
@@
 		(effects (font (face "Apple SD Gothic Neo") (size 2.5 2.5)) (justify left bottom))
 	)
-	(text "MLX90614 소자 1개는 FOV 안의 '평균'만 낸다. 그래서 2개를 다른 지점에 겨눠 공간 피크를 만든다."
+	(text "셀 IR 은 #1 한 존이고, #2 는 실온을 잰다 -> 발열값 = 표면온도 - 실온 (2026-09-25)."
 		(exclude_from_sim no)
 		(at 300.00 407.60 0)
 		(effects (font (face "Apple SD Gothic Neo") (size 2.0 2.0)) (justify left bottom))
 	)
-	(text "   temp_ir_surface = max(#1, #2)      temp_contact = max(DS18B20 #1, #2, #3)"
+	(text "   temp_ir_surface = #1      temp_contact = max(DS18B20 #1, #2, #3)      temp_ambient = #2 Ta"
 		(exclude_from_sim no)
 		(at 300.00 412.80 0)
@@
 		(effects (font (face "Apple SD Gothic Neo") (size 2.0 2.0)) (justify left bottom))
 	)
-	(text "[!] MLX90614 부착 거리 — 2cm 이내"
+	(text "[!] MLX90614 #1 부착 거리 — 2cm 이내"
 		(exclude_from_sim no)
 		(at 300.00 431.40 0)
